File: V2/Hw/Magspoof_V2/Magspoof_V2.kicad_pcb (KiCad board)
At the start: 2 copper layers, 35 x 20 mm, 24 parts, among them J1 USB_B_Micro, J2 SWD, J3 Coil, SW1 RST, SW2 S1, U1 AP2112K-3.3, U2 ATSAMD11C14A, U3 TC4424, U4 MCP73831

Commit message: Update desing
Parts:
- added D5: MBR120, Diode_SMD:D_SOD-123, B.Cu at (116.0, 105.2)
- moved G*** 1.01 mm to (130.8, 95.8)
Connections:
- BT1 pad 1: +BATT -> Net-(BT1-Pad1)
Routing:
- net +BATT: track 40.7 -> 33.8 mm
- net Net-(BT1-Pad1): track 0.00 -> 2.90 mm
Other:
- board text added: "+"
- board text added: "-"
- board text added: "Done"
- board text added: "Magspoof V3.1"
- board text removed: "Charged"
- board text removed: "Magspoof V2"
- board text removed: "V0.1"
Changed lines of the file:
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@@
   (general
     (thickness 1.6)
-    (drawings 18)
-    (tracks 276)
+    (drawings 19)
+    (tracks 268)
     (zones 0)
-    (modules 24)
-    (nets 28)
+    (modules 25)
+    (nets 29)
   )
   (page A4)
   (title_block
-    (title "Magspoof V2")
+    (title "Magspoof V3")
     (date 2019-08-26)
     (rev 0.1v)
@@
   )
   (layers
-    (0 F.Cu signal hide)
-    (31 B.Cu signal hide)
+    (0 F.Cu signal)
+    (31 B.Cu signal)
     (32 B.Adhes user)
     (33 F.Adhes user)
@@
       (outputformat 1)
       (mirror false)
-      (drillshape 1)
+      (drillshape 0)
       (scaleselection 1)
-      (outputdirectory ""))
+      (outputdirectory "/Users/eduardocontreras/Documents/Electronic_Cats/Proyectos/Hw/magspoof/V2/Hw/Magspoof_V2/gerber/"))
   )
   (net 0 "")
@@
   (net 26 "Net-(R3-Pad1)")
   (net 27 "Net-(R4-Pad1)")
+  (net 28 "Net-(BT1-Pad1)")
   (net_class Default "Esta es la clase de red por defecto."
     (clearance 0.25)
@@
     (add_net /Out_A)
     (add_net /Out_B)
+    (add_net "Net-(BT1-Pad1)")
+  )
+  (module Diode_SMD:D_SOD-123 (layer B.Cu)
+    (at 116.05 105.2 180)
+    (descr SOD-123)
+    (tags SOD-123)
+    (attr smd)
+    (fp_text reference D5 (at -3.45 0 180) (layer B.SilkS)
+      (effects (font (size 1 1) (thickness 0.15)) (justify mirror))
+    )
+    (fp_text value MBR120 (at 0 -2.1 180) (layer B.Fab)
+      (effects (font (size 1 1) (thickness 0.15)) (justify mirror))
+    )
+    (fp_line (start -2.25 1) (end 1.65 1) (layer B.SilkS) (width 0.12))
+    (fp_line (start -2.25 -1) (end 1.65 -1) (layer B.SilkS) (width 0.12))
+    (fp_line (start -2.35 1.15) (end -2.35 -1.15) (layer B.CrtYd) (width 0.05))
+    (fp_line (start 2.35 -1.15) (end -2.35 -1.15) (layer B.CrtYd) (width 0.05))
+    (fp_line (start 2.35 1.15) (end 2.35 -1.15) (layer B.CrtYd) (width 0.05))
+    (fp_line (start -2.35 1.15) (end 2.35 1.15) (layer B.CrtYd) (width 0.05))
+    (fp_line (start -1.4 0.9) (end 1.4 0.9) (layer B.Fab) (width 0.1))
+    (fp_line (start 1.4 0.9) (end 1.4 -0.9) (layer B.Fab) (width 0.1))
+    (fp_line (start 1.4 -0.9) (end -1.4 -0.9) (layer B.Fab) (width 0.1))
+    (fp_line (start -1.4 -0.9) (end -1.4 0.9) (layer B.Fab) (width 0.1))
+    (fp_line (start -0.75 0) (end -0.35 0) (layer B.Fab) (width 0.1))
+    (fp_line (start -0.35 0) (end -0.35 0.55) (layer B.Fab) (width 0.1))
+    (fp_line (start -0.35 0) (end -0.35 -0.55) (layer B.Fab) (width 0.1))
+    (fp_line (start -0.35 0) (end 0.25 0.4) (layer B.Fab) (width 0.1))
+    (fp_line (start 0.25 0.4) (end 0.25 -0.4) (layer B.Fab) (width 0.1))
+    (fp_line (start 0.25 -0.4) (end -0.35 0) (layer B.Fab) (width 0.1))
+    (fp_line (start 0.25 0) (end 0.75 0) (layer B.Fab) (width 0.1))
+    (fp_line (start -2.25 1) (end -2.25 -1) (layer B.SilkS) (width 0.12))
+    (fp_text user %R (at 0 2 180) (layer B.Fab)
+      (effects (font (size 1 1) (thickness 0.15)) (justify mirror))
+    )
+    (pad 2 smd rect (at 1.65 0 180) (size 0.9 1.2) (layers B.Cu B.Paste B.Mask)
+      (net 28 "Net-(BT1-Pad1)"))
+    (pad 1 smd rect (at -1.65 0 180) (size 0.9 1.2) (layers B.Cu B.Paste B.Mask)
+      (net 24 +BATT))
+    (model ${KISYS3DMOD}/Diode_SMD.3dshapes/D_SOD-123.wrl
+      (at (xyz 0 0 0))
+      (scale (xyz 1 1 1))
+      (rotate (xyz 0 0 0))
+    )
   )
   (module Aesthetics:electronic_cats_logo_4x3 (layer B.Cu)
-    (at 130.2 96.6 180)
+    (at 130.75 95.75 180)
     (fp_text reference G*** (at 0 0 180) (layer B.SilkS) hide
       (effects (font (size 1.524 1.524) (thickness 0.3)) (justify mirror))
@@
     (tags SOT-23-5)
     (attr smd)
-    (fp_text reference U4 (at 1.4 -2.9) (layer B.SilkS)
+    (fp_text reference U4 (at 3.5 -3.05) (layer B.SilkS)
       (effects (font (size 1 1) (thickness 0.15)) (justify mirror))
     )
@@
     (descr "Through hole straight pin header, 1x04, 2.54mm pitch, single row")
     (tags "Through hole pin header THT 1x04 2.54mm single row")
-    (fp_text reference J2 (at 0 -2.33 90) (layer F.SilkS)
+    (fp_text reference J2 (at 0 -2.71 180) (layer F.SilkS)
       (effects (font (size 1 1) (thickness 0.15)))
     )
@@
     (descr "Through hole straight pin header, 1x02, 2.54mm pitch, single row")
     (tags "Through hole pin header THT 1x02 2.54mm single row")
-    (fp_text reference BT1 (at 0 -2.33 90) (layer F.SilkS)
+    (fp_text reference BT1 (at -0.8 -2.8 180) (layer F.SilkS)
       (effects (font (size 1 1) (thickness 0.15)))
     )
@@
       (net 1 GND))
     (pad 1 thru_hole rect (at 0 0 90) (size 1.7 1.7) (drill 1) (layers *.Cu *.Mask)
-      (net 24 +BATT))
+      (net 28 "Net-(BT1-Pad1)"))
     (model ${KISYS3DMOD}/Connector_PinHeader_2.54mm.3dshapes/PinHeader_1x02_P2.54mm_Vertical.wrl
       (at (xyz 0 0 0))
@@
       (rotate (xyz 0 0 0))
     )
+  )
+  (gr_text - (at 118.9 106.55) (layer F.SilkS)
+    (effects (font (size 1 1) (thickness 0.15)))
+  )
+  (gr_text + (at 112.95 106.55) (layer F.SilkS)
+    (effects (font (size 1 1) (thickness 0.15)))
   )
   (gr_text Batt (at 116.8 102) (layer F.SilkS)
     (effects (font (size 1 1) (thickness 0.12)))
   )
-  (gr_text Charged (at 118.2 103.4) (layer F.SilkS)
+  (gr_text Done (at 117.25 103.4) (layer F.SilkS)
     (effects (font (size 1 1) (thickness 0.12)))
   )
-  (gr_text V0.1 (at 130 102.6) (layer B.SilkS)
-    (effects (font (size 1 1) (thickness 0.15)) (justify mirror))
-  )
-  (gr_text "Magspoof V2" (at 130 101) (layer B.SilkS)
+  (gr_text "Magspoof V3.1" (at 131.25 99.25) (layer B.SilkS)
     (effects (font (size 1 1) (thickness 0.15)) (justify mirror))
   )
@@
   (segment (start 116.65 98.9) (end 116.774999 98.775001) (width 0.5) (layer B.Cu) (net 24))
   (segment (start 116.65 100.7) (end 116.65 98.9) (width 0.5) (layer B.Cu) (net 24))
-  (via (at 136 101.5) (size 0.8) (drill 0.4) (layers F.Cu B.Cu) (net 24))
-  (segment (start 136.065 101.435) (end 136 101.5) (width 0.5) (layer F.Cu) (net 24))
-  (segment (start 137.7 101.435) (end 136.065 101.435) (width 0.5) (layer F.Cu) (net 24))
-  (segment (start 114.4 106.5) (end 114.4 108.1) (width 0.5) (layer B.Cu) (net 24))
-  (segment (start 115 105.9) (end 114.4 106.5) (width 0.5) (layer B.Cu) (net 24))
-  (segment (start 116.65 105.75) (end 116.8 105.9) (width 0.5) (layer B.Cu) (net 24))
-  (segment (start 116.65 100.7) (end 116.65 103.85) (width 0.5) (layer B.Cu) (net 24))
-  (segment (start 116.1 105.9) (end 116.65 105.35) (width 0.5) (layer B.Cu) (net 24))
-  (segment (start 115.9 105.9) (end 116.8 105.9) (width 0.5) (layer B.Cu) (net 24))
-  (segment (start 116.65 105.35) (end 116.65 105.75) (width 0.5) (layer B.Cu) (net 24))
-  (segment (start 115.9 105.9) (end 116.1 105.9) (width 0.5) (layer B.Cu) (net 24))
-  (segment (start 116.65 103.85) (end 116.65 105.35) (width 0.5) (layer B.Cu) (net 24))
-  (segment (start 115 105.9) (end 115.9 105.9) (width 0.5) (layer B.Cu) (net 24))
-  (segment (start 117.2 105.9) (end 116.65 105.35) (width 0.5) (layer B.Cu) (net 24))
-  (segment (start 117.6 105.9) (end 117.2 105.9) (width 0.5) (layer B.Cu) (net 24))
-  (segment (start 116.8 105.9) (end 117.6 105.9) (width 0.5) (layer B.Cu) (net 24))
-  (segment (start 117.6 105.9) (end 117.700002 106.000002) (width 0.5) (layer B.Cu) (net 24))
-  (segment (start 117.700002 106.000002) (end 135.099998 106.000002) (width 0.5) (layer B.Cu) (net 24))
-  (segment (start 136 105.1) (end 136 102.065685) (width 0.5) (layer B.Cu) (net 24))
-  (segment (start 135.099998 106.000002) (end 136 105.1) (width 0.5) (layer B.Cu) (net 24))
-  (segment (start 136 102.065685) (end 136 101.5) (width 0.5) (layer B.Cu) (net 24))
+  (segment (start 116.65 101.5) (end 116.65 100.7) (width 0.5) (layer B.Cu) (net 24))
+  (segment (start 116.65 103.05) (end 116.65 101.5) (width 0.5) (layer B.Cu) (net 24))
+  (segment (start 117.7 104.1) (end 116.65 103.05) (width 0.5) (layer B.Cu) (net 24))
+  (segment (start 117.7 105.2) (end 117.7 104.1) (width 0.5) (layer B.Cu) (net 24))
+  (segment (start 118.65 105.2) (end 119.75 106.3) (width 0.5) (layer B.Cu) (net 24))
+  (segment (start 117.7 105.2) (end 118.65 105.2) (width 0.5) (layer B.Cu) (net 24))
+  (segment (start 119.75 106.3) (end 134.9 106.3) (width 0.5) (layer B.Cu) (net 24))
+  (via (at 135.85 101.45) (size 0.8) (drill 0.4) (layers F.Cu B.Cu) (net 24))
+  (segment (start 135.85 105.35) (end 135.85 101.45) (width 0.5) (layer B.Cu) (net 24))
+  (segment (start 134.9 106.3) (end 135.85 105.35) (width 0.5) (layer B.Cu) (net 24))
+  (segment (start 137.685 101.45) (end 137.7 101.435) (width 0.5) (layer F.Cu) (net 24))
+  (segment (start 135.85 101.45) (end 137.685 101.45) (width 0.5) (layer F.Cu) (net 24))
   (via (at 118.575 103.25) (size 0.8) (drill 0.4) (layers F.Cu B.Cu) (net 25))
   (segment (start 116.45 103.25) (end 116.0625 103.6375) (width 0.3) (layer F.Cu) (net 25))
@@
   (segment (start 120.1 100.05) (end 120.8 100.05) (width 0.3) (layer B.Cu) (net 27))
   (segment (start 118.75 98.7) (end 120.1 100.05) (width 0.3) (layer B.Cu) (net 27))
+  (segment (start 114.4 105.2) (end 114.4 108.1) (width 0.5) (layer B.Cu) (net 28))
   (zone (net 1) (net_name GND) (layer F.Cu) (hatch edge 0.508)
     (connect_pads (clearance 0.508))
