File: V1/Hw/KiCad-PCB/MagSpoofTC.kicad_pcb (KiCad board)
At the start: 2 copper layers, 35 x 29 mm, 13 parts, among them IC1 ATTINY85-P, P1 - Battery +, P2 AVR ICSP, SW1 SW_PUSH, U1 TC4424

Commit message: footprint update
Other:
- net class Alimentacion removed
- net class Default removed
